File: DCDCv2/DCDCv2.kicad_sch (KiCad schematic)
At the start: 57 parts, among them M1 CSD18513Q5A, M1_2 CSD18513Q5A, M2 CSD18531Q5A, M3 CSD18533Q5A, M3_2 CSD18533Q5A, M4 CSD19534Q5A, M4_2 CSD19534Q5A, U1 LM5175PWPR

Commit message: added footprints and datasheets to some components
Parts:
- Cboot1, Cboot2, Css: footprint (none) -> Capacitor_SMD:C_0805_2012Metric_Pad1.18x1.45mm_HandSolder
- Cout_2, Cout_3, Cout_4: footprint (none) -> cap footprints:35SVPF82M
- M1, M3, M3_2, M4, M4_2: footprint (none) -> CSD18531Q5A footprint:8power tdfn
- M1_2, M2: footprint (none) -> CSD18531Q5A footprint:CSD18531Q5A
Connections:
- net 12 renamed sw1
- net 13 renamed rcs2
- net 19 renamed sw2
- net 26 renamed ldrv2
- net 28 renamed hdrv2
- net 31 renamed hdrv1
- net 7: no longer names the net of Cbias.1, Cout.1 (+), Cout_2.1 (+), Cout_3.1 (+), Cout_4.1 (+), Coutx.1, Coutx2.1, Coutx2_2.1, Coutx2_3.1, Coutx3.1, Coutx3_2.1, Coutx3_3.1, Coutx_2.1, Coutx_3.1, D3.2 (K), Iout.1 (+), M3.5 (Drain), M3.6 (Drain), M3.7 (Drain), M3.8 (Drain), M3.9 (Drain), M3_2.5 (Drain), M3_2.6 (Drain), M3_2.7 (Drain), M3_2.8 (Drain), M3_2.9 (Drain), Rfbt.1, U1.12 (VOSNS), U1.24 (BIAS)
- net 9 renamed ldrv1

Commit message: specced more components and added some cap footprints
Parts:
- Cbulk: footprint (none) -> cap footprints:PCAP_6.3x7.7-ELECT_NCA
- Cf: footprint (none) -> Capacitor_SMD:C_0603_1608Metric_Pad1.08x0.95mm_HandSolder
- Cin, Cin_2, Cin_5: footprint (none) -> cap footprints:PCAP_SVP_E12_PAN
- Df: footprint (none) -> Diode_SMD:D_SMC
- Rf: footprint (none) -> Resistor_SMD:R_0603_1608Metric_Pad0.98x0.95mm_HandSolder
Changed lines of the file:
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@@
 			)
 		)
-		(property "Footprint" ""
+		(property "Footprint" "cap footprints:PCAP_SVP_E12_PAN"
 			(at 97.79 72.39 0)
 			(effects
@@
 			)
 		)
-		(property "Datasheet" ""
+		(property "Datasheet" "https://industrial.panasonic.com/ww/products/pt/os-con/models/50SVPF39M"
 			(at 97.79 72.39 0)
 			(effects
@@
 			)
 		)
-		(property "Footprint" ""
+		(property "Footprint" "cap footprints:PCAP_SVP_E12_PAN"
 			(at 115.57 72.39 0)
 			(effects
@@
 			)
 		)
-		(property "Datasheet" ""
+		(property "Datasheet" "https://industrial.panasonic.com/ww/products/pt/os-con/models/50SVPF39M"
 			(at 115.57 72.39 0)
 			(effects
@@
 			)
 		)
-		(property "Footprint" ""
+		(property "Footprint" "Capacitor_SMD:C_0603_1608Metric_Pad1.08x0.95mm_HandSolder"
 			(at 289.56 100.33 0)
 			(effects
@@
 			)
 		)
-		(property "Datasheet" ""
+		(property "Datasheet" "https://product.tdk.com/system/files/dam/doc/product/capacitor/ceramic/mlcc/catalog/mlcc_commercial_general_en.pdf"
 			(at 289.56 100.33 0)
 			(effects
@@
 			)
 		)
-		(property "Footprint" ""
+		(property "Footprint" "Diode_SMD:D_SMC"
 			(at 289.56 46.99 0)
 			(effects
@@
 			)
 		)
-		(property "Datasheet" ""
+		(property "Datasheet" "https://www.vishay.com/docs/88742/sl42.pdf"
 			(at 289.56 46.99 0)
 			(effects
@@
 			)
 		)
-		(property "Footprint" ""
+		(property "Footprint" "cap footprints:PCAP_SVP_E12_PAN"
 			(at 168.91 72.39 0)
 			(effects
@@
 			)
 		)
-		(property "Datasheet" ""
+		(property "Datasheet" "https://industrial.panasonic.com/ww/products/pt/os-con/models/50SVPF39M"
 			(at 168.91 72.39 0)
 			(effects
@@
 			)
 		)
-		(property "Footprint" ""
+		(property "Footprint" "Resistor_SMD:R_0603_1608Metric_Pad0.98x0.95mm_HandSolder"
 			(at 289.56 69.85 0)
 			(effects
@@
 			)
 		)
-		(property "Datasheet" ""
+		(property "Datasheet" "https://www.yageo.com/upload/media/product/products/datasheet/rchip/PYu-RC_Group_51_RoHS_L_12.pdf"
 			(at 289.56 69.85 0)
 			(effects
@@
 			)
 		)
-		(property "Footprint" ""
+		(property "Footprint" "cap footprints:PCAP_6.3x7.7-ELECT_NCA"
 			(at 71.12 72.39 0)
 			(effects
@@
 			)
 		)
-		(property "Datasheet" ""
+		(property "Datasheet" "https://www.nichicon.co.jp/english/series_items/catalog_pdf/e-uud.pdf"
 			(at 71.12 72.39 0)
 			(effects

Commit message: specced more components (dec 29 2024)
Parts:
- removed Iout: WB_CURRENT_LOAD, symbol DCDCv2-altium-import:root_3_Iout
- removed Vin: WB_BATTERY, symbol DCDCv2-altium-import:root_3_Vin
- added J1, J2: Screw_Terminal_01x02, screwterm footprint:CONN_1777545, symbol Connector:Screw_Terminal_01x02
- Cbias, Cslope: footprint (none) -> Capacitor_SMD:C_0603_1608Metric_Pad1.08x0.95mm_HandSolder
- Ccomp: footprint (none) -> Capacitor_SMD:C_0805_2012Metric_Pad1.18x1.45mm_HandSolder
- Ccomp2: footprint (none) -> Capacitor_SMD:C_0402_1005Metric_Pad0.74x0.62mm_HandSolder
- Cout: footprint (none) -> cap footprints:35SVPF82M
- Coutx, Coutx2_2, Coutx2_3, Coutx3, Coutx3_2, Coutx3_3, Coutx_2, Coutx_3: footprint (none) -> Capacitor_SMD:C_1210_3225Metric_Pad1.33x2.70mm_HandSolder
Connections:
- net 0: now also J1.2 (Pin_2), J2.2 (Pin_2)
- net at Cbulk.1 (+), Cin.1 (+), Cin_2.1 (+)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: now also J1.1 (Pin_1)
- net at Cbias.1, Cout.1 (+), Cout_2.1 (+)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: now also J2.1 (Pin_1)

Commit message: finished speccing components in schematic
Parts:
- Ccs1: renamed from Ccs; footprint (none) -> Capacitor_SMD:C_0603_1608Metric_Pad1.08x0.95mm_HandSolder
- Cin_3, Cin_4: footprint (none) -> cap footprints:35SVPF82M
- Cvcc1: renamed from Cvcc; footprint (none) -> Capacitor_SMD:C_0603_1608Metric_Pad1.08x0.95mm_HandSolder
- D2, Dboot1, Dboot2: footprint (none) -> Diode_SMD:D_SMC_Handsoldering
- D3: footprint (none) -> Package_TO_SOT_SMD:TO-252-2
- Df1: renamed from Df; footprint Diode_SMD:D_SMC -> Diode_SMD:D_SMC_Handsoldering
- L1: footprint (none) -> Inductor_THT_Wurth:L_Wurth_WE-HCFT-3521; ALTIUM_VALUE 4.065uH -> 2.2uH
- Rcomp1: renamed from Rcomp; footprint (none) -> Resistor_SMD:R_0603_1608Metric_Pad0.98x0.95mm_HandSolder
- Rcsg1: renamed from Rcsg; footprint (none) -> Resistor_SMD:R_0603_1608Metric_Pad0.98x0.95mm_HandSolder
- Rcsp1: renamed from Rcsp; footprint (none) -> Resistor_SMD:R_0603_1608Metric_Pad0.98x0.95mm_HandSolder
- Rfbb1: renamed from Rfbb; footprint (none) -> Resistor_SMD:R_0603_1608Metric_Pad0.98x0.95mm_HandSolder
- Rmode1: renamed from Rmode; footprint (none) -> Resistor_SMD:R_0603_1608Metric_Pad0.98x0.95mm_HandSolder
- Rpg1: renamed from Rpg; footprint (none) -> Resistor_SMD:R_0603_1608Metric_Pad0.98x0.95mm_HandSolder
- Rsense1: renamed from Rsense; footprint (none) -> Rsense footprint:RES_WSLP3921_.002OHM_VIS; ALTIUM_VALUE 2.394m -> 2.5m
- Rt1: renamed from Rt; footprint (none) -> Resistor_SMD:R_0603_1608Metric_Pad0.98x0.95mm_HandSolder
- Ruvb1: renamed from Ruvb; footprint (none) -> Resistor_SMD:R_0603_1608Metric_Pad0.98x0.95mm_HandSolder
- Ruvt1: renamed from Ruvt; footprint (none) -> Resistor_SMD:R_0603_1608Metric_Pad0.98x0.95mm_HandSolder
- U1: footprint (none) -> LM5175:PWP0028F_N
- renumbered Cbias to Cbias1, Cbulk to Cbulk1, Ccomp to Ccomp1, Cf to Cf1, Cin to Cin1, Cout to Cout1, Coutx to Coutx1, Cslope to Cslope1, Css to Css1, Rf to Rf1, Rfbt to Rfbt1, J1 to Vin1, J2 to Vout1
Connections:
- net 0 renamed GND

Commit message: preliminary pcb layout finished
Parts:
- Cbulk1: footprint cap footprints:PCAP_6.3x7.7-ELECT_NCA -> cap footprints:CAPAE660X800N
- Cin_3, Cin_4: footprint cap footprints:35SVPF82M -> cap footprints:PCAP_SVP_E12_PAN
- Coutx2: footprint (none) -> Capacitor_SMD:C_1210_3225Metric_Pad1.33x2.70mm_HandSolder
- M1_2, M2: footprint CSD18531Q5A footprint:CSD18531Q5A -> CSD18531Q5A footprint:8power tdfn
- Rfbt1: footprint (none) -> Resistor_SMD:R_0603_1608Metric_Pad0.98x0.95mm_HandSolder
Connections:
- net Vin: now reaches Cbulk1.1 (+), Cin1.1 (+), Cin_2.1 (+), Cin_3.1 (+), Cin_4.1 (+), Cin_5.1 (+), Df1.2 (A), M1.5 (Drain), M1.6 (Drain), M1.7 (Drain), M1.8 (Drain), M1.9 (Drain), M1_2.5 (Drain), M1_2.6 (Drain), M1_2.7 (Drain), M1_2.8 (Drain), M1_2.9 (Drain), Ruvt1.1, U1.3 (VINSNS), Vin1.1 (Pin_1)
- net Vout: now reaches Cbias1.1, Cout1.1 (+), Cout_2.1 (+), Cout_3.1 (+), Cout_4.1 (+), Coutx1.1, Coutx2.1, Coutx2_2.1, Coutx2_3.1, Coutx3.1, Coutx3_2.1, Coutx3_3.1, Coutx_2.1, Coutx_3.1, D3.2 (K), M3.5 (Drain), M3.6 (Drain), M3.7 (Drain), M3.8 (Drain), M3.9 (Drain), M3_2.5 (Drain), M3_2.6 (Drain), M3_2.7 (Drain), M3_2.8 (Drain), M3_2.9 (Drain), Rfbt1.1, U1.12 (VOSNS), U1.24 (BIAS), Vout1.1 (Pin_1)
Changed lines of the file:
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@@
 	)
 	(junction
+		(at 1037.59 27.94)
+		(diameter 0)
+		(color 0 0 0 0)
+	)
+	(junction
 		(at 419.1 266.7)
 		(diameter 0)
@@
 	(wire
 		(pts
-			(xy 44.45 67.31) (xy 44.45 27.94)
-		)
-		(stroke
-			(width 0)
-			(type default)
-		)
-	)
-	(wire
-		(pts
 			(xy 179.07 326.39) (xy 179.07 255.27)
 		)
@@
 	(wire
 		(pts
+			(xy 44.45 27.94) (xy 44.45 67.31)
+		)
+		(stroke
+			(width 0)
+			(type default)
+		)
+	)
+	(wire
+		(pts
 			(xy 375.92 152.4) (xy 920.75 152.4)
 		)
@@
 			)
 		)
-		(property "Footprint" "cap footprints:35SVPF82M"
+		(property "Footprint" "cap footprints:PCAP_SVP_E12_PAN"
 			(at 133.35 72.39 0)
 			(effects
@@
 					(size 1.27 1.27)
 				)
-				(hide yes)
 			)
 		)
@@
 			)
 		)
-		(property "Footprint" "cap footprints:35SVPF82M"
+		(property "Footprint" "cap footprints:PCAP_SVP_E12_PAN"
 			(at 151.13 72.39 0)
 			(effects
@@
 	(symbol
 		(lib_id "power:PWR_FLAG")
+		(at 71.12 27.94 0)
+		(unit 1)
+		(exclude_from_sim no)
+		(in_bom yes)
+		(on_board yes)
+		(dnp no)
+		(fields_autoplaced yes)
+		(property "Reference" "#FLG09"
+			(at 71.12 26.035 0)
+			(effects
+				(font
+					(size 1.27 1.27)
+				)
+				(hide yes)
+			)
+		)
+		(property "Value" "PWR_FLAG"
+			(at 71.12 22.86 0)
+			(effects
+				(font
+					(size 1.27 1.27)
+				)
+			)
+		)
+		(property "Footprint" ""
+			(at 71.12 27.94 0)
+			(effects
+				(font
+					(size 1.27 1.27)
+				)
+				(hide yes)
+			)
+		)
+		(property "Datasheet" "~"
+			(at 71.12 27.94 0)
+			(effects
+				(font
+					(size 1.27 1.27)
+				)
+				(hide yes)
+			)
+		)
+		(property "Description" "Special symbol for telling ERC where power comes from"
+			(at 71.12 27.94 0)
+			(effects
+				(font
+					(size 1.27 1.27)
+				)
+				(hide yes)
+			)
+		)
+		(pin "1"
+		)
+		(instances
+			(project ""
+				(path "/83b78cfd-fb8d-4c5f-85af-30e619b5f1da"
+					(reference "#FLG09")
+					(unit 1)
+				)
+			)
+		)
+	)
+	(symbol
+		(lib_id "power:+1V0")
+		(at 44.45 27.94 0)
+		(unit 1)
+		(exclude_from_sim no)
+		(in_bom yes)
+		(on_board yes)
+		(dnp no)
+		(fields_autoplaced yes)
+		(property "Reference" "#PWR01"
+			(at 44.45 31.75 0)
+			(effects
+				(font
+					(size 1.27 1.27)
+				)
+				(hide yes)
+			)
+		)
+		(property "Value" "Vin"
+			(at 44.45 22.86 0)
+			(effects
+				(font
+					(size 1.27 1.27)
+				)
+			)
+		)
+		(property "Footprint" ""
+			(at 44.45 27.94 0)
+			(effects
+				(font
+					(size 1.27 1.27)
+				)
+				(hide yes)
+			)
+		)
+		(property "Datasheet" ""
+			(at 44.45 27.94 0)
+			(effects
+				(font
+					(size 1.27 1.27)
+				)
+				(hide yes)
+			)
+		)
+		(property "Description" "Power symbol creates a global label with name \"+1V0\""
+			(at 44.45 27.94 0)
+			(effects
+				(font
+					(size 1.27 1.27)
+				)
+				(hide yes)
+			)
+		)
+		(pin "1"
+		)
+		(instances
+			(project ""
+				(path "/83b78cfd-fb8d-4c5f-85af-30e619b5f1da"
+					(reference "#PWR01")
+					(unit 1)
+				)
+			)
+		)
+	)
+	(symbol
+		(lib_id "power:PWR_FLAG")
 		(at 369.57 198.12 0)
 		(unit 1)
@@
 			)
 		)
-		(property "Footprint" ""
+		(property "Footprint" "Capacitor_SMD:C_1210_3225Metric_Pad1.33x2.70mm_HandSolder"
 			(at 740.41 67.31 0)
 			(effects
@@
 			)
 		)
-		(property "Datasheet" ""
+		(property "Datasheet" "https://mm.digikey.com/Volume0/opasdata/d220001/medias/docus/41/CL32B106KBJNNNE_Spec.pdf"
 			(at 740.41 67.31 0)
 			(effects
@@
 			)
 		)
-		(property "Footprint" ""
+		(property "Footprint" "Resistor_SMD:R_0603_1608Metric_Pad0.98x0.95mm_HandSolder"
 			(at 652.78 50.8 0)
 			(effects
@@
 			)
 		)
-		(property "Datasheet" ""
+		(property "Datasheet" "https://www.yageo.com/upload/media/product/products/datasheet/rchip/PYu-RC_Group_51_RoHS_L_12.pdf"
 			(at 652.78 50.8 0)
 			(effects
@@
 			)
 		)
-		(property "Footprint" "CSD18531Q5A footprint:CSD18531Q5A"
+		(property "Footprint" "CSD18531Q5A footprint:8power tdfn"
 			(at 394.97 97.79 0)
 			(effects
@@
 	)
 	(symbol
+		(lib_id "power:+1V0")
+		(at 1037.59 27.94 0)
+		(unit 1)
+		(exclude_from_sim no)
+		(in_bom yes)
+		(on_board yes)
+		(dnp no)
+		(fields_autoplaced yes)
+		(property "Reference" "#PWR013"
+			(at 1037.59 31.75 0)
+			(effects
+				(font
+					(size 1.27 1.27)
+				)
+				(hide yes)
+			)
+		)
+		(property "Value" "Vout"
+			(at 1037.59 22.86 0)
+			(effects
+				(font
+					(size 1.27 1.27)
+				)
+			)
+		)
+		(property "Footprint" ""
+			(at 1037.59 27.94 0)
+			(effects
+				(font
+					(size 1.27 1.27)
+				)
+				(hide yes)
+			)
+		)
+		(property "Datasheet" ""
+			(at 1037.59 27.94 0)
+			(effects
+				(font
+					(size 1.27 1.27)
+				)
+				(hide yes)
+			)
+		)
+		(property "Description" "Power symbol creates a global label with name \"+1V0\""
+			(at 1037.59 27.94 0)
+			(effects
+				(font
+					(size 1.27 1.27)
+				)
+				(hide yes)
+			)
+		)
+		(pin "1"
+		)
+		(instances
+			(project ""
+				(path "/83b78cfd-fb8d-4c5f-85af-30e619b5f1da"
+					(reference "#PWR013")
+					(unit 1)
+				)
+			)
+		)
+	)
+	(symbol
 		(lib_id "DCDCv2-altium-import:root_1_Cout")
 		(at 957.58 68.58 0)
@@
 			)
 		)
-		(property "Footprint" "cap footprints:PCAP_6.3x7.7-ELECT_NCA"
+		(property "Footprint" "cap footprints:CAPAE660X800N"
 			(at 71.12 72.39 0)
 			(effects
@@
 			)
 		)
-		(property "Footprint" "CSD18531Q5A footprint:CSD18531Q5A"
+		(property "Footprint" "CSD18531Q5A footprint:8power tdfn"
 			(at 412.75 43.18 0)
 			(effects

Commit message: finished PCB layout
Connections:
- net GND: no longer U1.10 (AGND), U1.22 (PGND), U1.29 (PAD)
- new net GNDA: U1.10 (AGND), U1.22 (PGND), U1.29 (PAD)
Other:
- moved on the sheet: D2, M3_2
