File: DCDCv2/DCDCv2.kicad_pcb (KiCad board)
At the start: 2 copper layers, 49 parts, among them M1 CSD18513Q5A, M3 CSD18533Q5A, M3_2 CSD18533Q5A, M4 CSD19534Q5A, M4_2 CSD19534Q5A, U1 LM5175PWPR

Commit message: preliminary pcb layout finished
Parts:
- added Cbulk1: UUD1V680MCL1GS, cap footprints:CAPAE660X800N, F.Cu at (80.2, 59.9)
- added Cin1: 50SVPF39M, cap footprints:PCAP_SVP_E12_PAN, F.Cu at (50.2, 60.0)
- added Cin_2: 50SVPF39M, cap footprints:PCAP_SVP_E12_PAN, F.Cu at (40.2, 60.0)
- added Cin_5: 50SVPF39M, cap footprints:PCAP_SVP_E12_PAN, F.Cu at (60.2, 60.0)
- added Coutx2: C5750X7R2E684M, Capacitor_SMD:C_1210_3225Metric_Pad1.33x2.70mm_HandSolder, B.Cu at (107.2, 59.5)
- added G***: LOGO, logo:logo, F.Cu at (32.5, 92.0)
- added M1_2: CSD18513Q5A, CSD18531Q5A footprint:8power tdfn, F.Cu at (75.6, 75.2)
- added M2: CSD18531Q5A, CSD18531Q5A footprint:8power tdfn, F.Cu at (84.3, 78.7)
- added Rfbt1: RC0603FR-07576KL, Resistor_SMD:R_0603_1608Metric_Pad0.98x0.95mm_HandSolder, F.Cu at (86.2, 51.0)
- Cin_3, Cin_4: footprint cap footprints:35SVPF82M -> cap footprints:PCAP_SVP_E12_PAN
- Coutx1, Coutx2_2, Coutx2_3, Coutx3, Coutx3_2, Coutx3_3, Coutx_2, Coutx_3, D2, D3, Df1: moved to B.Cu
- moved Cout_4 77.0 mm to (140.2, 59.5), turned to 90 degrees
- moved Ruvt1 71.5 mm to (83.6, 32.5), turned to 180 degrees
- moved Ruvb1 69.4 mm to (79.2, 32.5), turned to 180 degrees
- moved Rf1 68.8 mm to (91.2, 33.0), turned to -90 degrees
- moved Cf1 67.3 mm to (93.2, 33.0), turned to 90 degrees
- moved Cvcc1 64.7 mm to (105.5, 44.7)
- moved Css1 64.5 mm to (83.2, 41.2), turned to 180 degrees
- moved Cout_3 63.6 mm to (130.1, 59.5), turned to 90 degrees
- moved Vin1 63.5 mm to (25.5, 79.8), turned to -90 degrees
- moved Cbias1 62.6 mm to (103.2, 36.0)
- moved Rt1 62.5 mm to (82.8, 36.5), turned to 180 degrees
- moved Cslope1 62.5 mm to (83.2, 39.0), turned to 180 degrees
- moved Rmode1 59.5 mm to (82.8, 34.5), turned to 180 degrees
- moved Ccomp1 59.3 mm to (81.6, 44.2), turned to 180 degrees
- moved Cboot1 59.1 mm to (98.8, 35.0), turned to 180 degrees
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Connections:
- Cbias1 pad 1: Net-(Cout1-+) -> Vout
- Cin_3 pad 1: Net-(Cbulk1-+) -> Vin
- Cin_4 pad 1: Net-(Cbulk1-+) -> Vin
- Cout1 pad 1: Net-(Cout1-+) -> Vout
- Cout_2 pad 1: Net-(Cout1-+) -> Vout
- Cout_3 pad 1: Net-(Cout1-+) -> Vout
- Cout_4 pad 1: Net-(Cout1-+) -> Vout
- Coutx1 pad 1: Net-(Cout1-+) -> Vout
- Coutx2_2 pad 1: Net-(Cout1-+) -> Vout
- Coutx2_3 pad 1: Net-(Cout1-+) -> Vout
- Coutx3 pad 1: Net-(Cout1-+) -> Vout
- Coutx3_2 pad 1: Net-(Cout1-+) -> Vout
- Coutx3_3 pad 1: Net-(Cout1-+) -> Vout
- Coutx_2 pad 1: Net-(Cout1-+) -> Vout
- Coutx_3 pad 1: Net-(Cout1-+) -> Vout
- D3 pad 2: Net-(Cout1-+) -> Vout
- Df1 pad 2: Net-(Cbulk1-+) -> Vin
- M1 pad 5: Net-(Cbulk1-+) -> Vin
- M3 pad 5: Net-(Cout1-+) -> Vout
- M3_2 pad 5: Net-(Cout1-+) -> Vout
- Ruvt1 pad 1: Net-(Cbulk1-+) -> Vin
- U1 pad 12: Net-(Cout1-+) -> Vout
- U1 pad 24: Net-(Cout1-+) -> Vout
- U1 pad 3: Net-(Cbulk1-+) -> Vin
- Vin1 pad 1: Net-(Cbulk1-+) -> Vin
- Vout1 pad 1: Net-(Cout1-+) -> Vout
Routing:
- net /sw2: track 0.00 -> 88.0 mm, vias 0 -> 66
- net Vout: track 0.00 -> 70.5 mm, vias 0 -> 99
- net /hdrv1: track 0.00 -> 68.8 mm, vias 0 -> 3
- net /hdrv2: track 0.00 -> 56.5 mm, vias 0 -> 3
- net /ldrv1: track 0.00 -> 55.5 mm, vias 0 -> 2
- net /sw1: track 0.00 -> 54.8 mm, vias 0 -> 98
- net /ldrv2: track 0.00 -> 54.1 mm, vias 0 -> 3
- net Vin: track 0.00 -> 44.4 mm, vias 0 -> 97
- net GND: track 0.00 -> 33.1 mm, vias 0 -> 380
- net Net-(Dboot1-A): track 0.00 -> 30.0 mm, vias 0 -> 2
- net Net-(Df1-K): track 0.00 -> 29.3 mm, vias 0 -> 1
- net Net-(Dboot1-K): track 0.00 -> 29.0 mm
- net /rcs2: track 0.00 -> 17.9 mm, vias 0 -> 18
- net Net-(Dboot2-K): track 0.00 -> 17.8 mm
- net Net-(U1-EN): track 0.00 -> 13.4 mm
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- added copper zone on B.Cu, net /rcs2
- added copper zone on F.Cu, net /rcs2
- added copper zone on B.Cu, net /sw1
- added copper zone on F.Cu, net /sw1
- added copper zone on In1.Cu, net /sw1
- added copper zone on In2.Cu, net /sw1
- added copper zone on B.Cu, net /sw2
- added copper zone on F.Cu, net /sw2
- added copper zone on In1.Cu, net /sw2
- added copper zone on In2.Cu, net /sw2
- added copper zone on B.Cu, net GND
- added copper zone on F.Cu, net GND
- added copper zone on In1.Cu, net GND
- added copper zone on In2.Cu, net GND
- added copper zone on B.Cu, net Vin
- added copper zone on F.Cu, net Vin
- added copper zone on In1.Cu, net Vin
- added copper zone on In2.Cu, net Vin
- added copper zone on B.Cu, net Vout
- added copper zone on F.Cu, net Vout
- added copper zone on In1.Cu, net Vout
- added copper zone on In2.Cu, net Vout
Other:
- board outline added: 137.2 x 79 mm
- copper layers 2 -> 4
- board text added: "FCP 24V 20A DC/DC CONVERTER"
- board text added: "Timothy Kwan"
- board text added: "{dblquote}PISSMAN 8{dblquote}"

Commit message: added 3d models for capacitors
Parts:
- moved G*** 19.2 mm to (51.5, 89.5)
Changed lines of the file:
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@@
 			(pintype "passive")
 		)
+		(model "${KIPRJMOD}/cap footprints.pretty/8 SIZE CODE E12.stp"
+			(offset
+				(xyz 0 0 0)
+			)
+			(scale
+				(xyz 1 1 1)
+			)
+			(rotate
+				(xyz -90 0 90)
+			)
+		)
 	)
 	(footprint "screwterm footprint:CONN_1777545"
@@
 			(pintype "passive")
 		)
+		(model "${KIPRJMOD}/cap footprints.pretty/8 SIZE CODE E12.stp"
+			(offset
+				(xyz 0 0 0)
+			)
+			(scale
+				(xyz 1 1 1)
+			)
+			(rotate
+				(xyz -90 0 90)
+			)
+		)
 	)
 	(footprint "Capacitor_SMD:C_0603_1608Metric_Pad1.08x0.95mm_HandSolder"
@@
 			(pintype "passive")
 		)
+		(model "${KIPRJMOD}/cap footprints.pretty/8 SIZE CODE E12.stp"
+			(offset
+				(xyz 0 0 0)
+			)
+			(scale
+				(xyz 1 1 1)
+			)
+			(rotate
+				(xyz -90 0 90)
+			)
+		)
 	)
 	(footprint "Diode_SMD:D_SMC_Handsoldering"
@@
 			(pintype "passive")
 		)
+		(model "${KIPRJMOD}/cap footprints.pretty/8 SIZE CODE E12.stp"
+			(offset
+				(xyz 0 0 0)
+			)
+			(scale
+				(xyz 1 1 1)
+			)
+			(rotate
+				(xyz -90 0 90)
+			)
+		)
 	)
 	(footprint "Capacitor_SMD:C_0603_1608Metric_Pad1.08x0.95mm_HandSolder"
@@
 			(pintype "passive")
 		)
+		(model "${KIPRJMOD}/cap footprints.pretty/8 SIZE CODE E12.stp"
+			(offset
+				(xyz 0 0 0)
+			)
+			(scale
+				(xyz 1 1 1)
+			)
+			(rotate
+				(xyz -90 0 90)
+			)
+		)
 	)
 	(footprint "Inductor_THT_Wurth:L_Wurth_WE-HCFT-3521"
@@
 		)
 		(model "UUD1V680MCL1GS.stp"
+			(hide yes)
+			(offset
+				(xyz 0 0 0)
+			)
+			(scale
+				(xyz 1 1 1)
+			)
+			(rotate
+				(xyz 0 0 0)
+			)
+		)
+		(model "${KIPRJMOD}/cap footprints.pretty/PCAP_6_3x7_7-ELECT_NCA.step"
 			(offset
 				(xyz 0 0 0)
@@
 			(pintype "passive")
 		)
+		(model "${KIPRJMOD}/cap footprints.pretty/8 SIZE CODE E12.stp"
+			(offset
+				(xyz 0 0 0)
+			)
+			(scale
+				(xyz 1 1 1)
+			)
+			(rotate
+				(xyz -90 0 90)
+			)
+		)
 	)
 	(footprint "screwterm footprint:CONN_1777545"
@@
 			(pintype "passive")
 		)
+		(model "${KIPRJMOD}/cap footprints.pretty/8 SIZE CODE E12.stp"
+			(offset
+				(xyz 0 0 0)
+			)
+			(scale
+				(xyz 1 1 1)
+			)
+			(rotate
+				(xyz -90 0 90)
+			)
+		)
 	)
 	(footprint "CSD18531Q5A footprint:8power tdfn"
@@
 			(layer "F.Fab")
 		)
-		(fp_text user "LM5175"
-			(at -0.999999 6.000001 0)
+		(fp_text user "Designator4"
+			(at -3.81 -6.223 0)
 			(unlocked yes)
 			(layer "F.SilkS")
@@
 			)
 		)
-		(fp_text user "Designator4"
-			(at -3.81 -6.223 0)
+		(fp_text user "LM5175"
+			(at -0.999999 6.000001 0)
 			(unlocked yes)
 			(layer "F.SilkS")
@@
 			(pintype "passive")
 		)
+		(model "${KIPRJMOD}/cap footprints.pretty/8 SIZE CODE E12.stp"
+			(offset
+				(xyz 0 0 0)
+			)
+			(scale
+				(xyz 1 1 1)
+			)
+			(rotate
+				(xyz -90 0 90)
+			)
+		)
 	)
 	(footprint "Resistor_SMD:R_0603_1608Metric_Pad0.98x0.95mm_HandSolder"
@@
 			(pintype "passive")
 		)
+		(model "${KIPRJMOD}/cap footprints.pretty/8 SIZE CODE E12.stp"
+			(offset
+				(xyz 0 0 0)
+			)
+			(scale
+				(xyz 1 1 1)
+			)
+			(rotate
+				(xyz -90 0 90)
+			)
+		)
 	)
 	(footprint "Diode_SMD:D_SMC_Handsoldering"
@@
 	(footprint "logo:logo"
 		(layer "F.Cu")
-		(at 32.5 92)
+		(at 51.5 89.5)
 		(property "Reference" "G***"
 			(at 0 0 0)
@@
 		(fp_poly
 			(pts
-				(xy -4.73 3.14) (xy -4.97 3.47) (xy -4.49 3.47) (xy -4.73 3.14)
+				(xy -5.04 3.14) (xy -5.38 3.61) (xy -4.7 3.61) (xy -5.04 3.14)
 			)
 			(stroke
@@
 	)
 	(gr_text "FCP 24V 20A DC/DC CONVERTER"
-		(at 21 99 0)
+		(at 117 89.5 0)
 		(layer "F.SilkS")
 		(effects
@@
 	)
 	(gr_text "Timothy Kwan\n\n\n"
-		(at 21.5 110.5 0)
+		(at 117.5 101 0)
 		(layer "F.SilkS")
 		(effects
@@
 	)
 	(gr_text "{dblquote}PISSMAN 8{dblquote} "
-		(at 21 102.5 0)
+		(at 117 93 0)
 		(layer "F.SilkS")
 		(effects
@@
 		(layer "F.Cu")
 		(hatch edge 0.5)
+		(connect_pads
+			(clearance 0)
+		)
+		(min_thickness 0.25)
+		(filled_areas_thickness no)
+		(keepout
+			(tracks allowed)
+			(vias allowed)
+			(pads allowed)
+			(copperpour not_allowed)
+			(footprints allowed)
+		)
+		(fill
+			(thermal_gap 0.5)
+			(thermal_bridge_width 0.5)
+		)
+		(polygon
+			(pts
+				(xy 96 63) (xy 96.5 63) (xy 96.5 64) (xy 96 64)
+			)
+		)
+	)
+	(zone
+		(net 0)
+		(net_name "")
+		(layer "F.Cu")
+		(hatch edge 0.5)
 		(connect_pads yes
 			(clearance 0)
@@
 		(polygon
 			(pts
-				(xy 98.25 59) (xy 99.25 59) (xy 99.25 55.5) (xy 97.75 54) (xy 97.75 53) (xy 97.25 53) (xy 97.25 55)
+				(xy 98.25 59) (xy 99.25 59) (xy 99.25 55.5) (xy 98.25 54) (xy 98.25 52) (xy 96.75 52) (xy 96.75 55)
 				(xy 98.25 56)
 			)

Commit message: not much changed since last commit
Parts:
- moved G*** 12.8 mm to (39.5, 94.0)
Routing:
- net /hdrv2: track 56.5 -> 54.6 mm
Other:
- board text added: "ok"
- board text removed: "{dblquote}PISSMAN 8{dblquote}"
Changed lines of the file:
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@@
 	(footprint "logo:logo"
 		(layer "F.Cu")
-		(at 51.5 89.5)
+		(at 39.5 94)
 		(property "Reference" "G***"
 			(at 0 0 0)
@@
 		)
 	)
-	(gr_text "{dblquote}PISSMAN 8{dblquote} "
+	(gr_text "ok\n"
 		(at 117 93 0)
 		(layer "F.SilkS")
@@
 		(net 1)
 	)
-	(via micro
+	(via
 		(at 92.775 43.5)
 		(size 0.6)
@@
 		(net 1)
 	)
-	(via micro
+	(via
 		(at 94.775 43.5)
 		(size 0.6)
@@
 		(net 1)
 	)
-	(via micro
+	(via
 		(at 93.775 41.5)
 		(size 0.6)
@@
 		(net 1)
 	)
-	(via micro
+	(via
 		(at 93.775 39.5)
 		(size 0.6)
@@
 		(net 1)
 	)
-	(via micro
+	(via
 		(at 93.775 43.5)
 		(size 0.6)
@@
 		(net 1)
 	)
-	(via micro
+	(via
 		(at 92.775 42.5)
 		(size 0.6)
@@
 		(net 1)
 	)
-	(via micro
+	(via
 		(at 93.775 40.5)
 		(size 0.6)
@@
 		(net 1)
 	)
-	(via micro
+	(via
 		(at 94.775 41.5)
 		(size 0.6)
@@
 		(net 1)
 	)
-	(via micro
+	(via
 		(at 92.775 39.5)
 		(size 0.6)
@@
 		(net 1)
 	)
-	(via micro
+	(via
 		(at 92.775 41.5)
 		(size 0.6)
@@
 		(net 1)
 	)
-	(via micro
+	(via
 		(at 93.775 42.5)
 		(size 0.6)
@@
 		(net 1)
 	)
-	(via micro
+	(via
 		(at 94.775 42.5)
 		(size 0.6)
@@
 		(net 1)
 	)
-	(via micro
+	(via
 		(at 92.775 40.5)
 		(size 0.6)
@@
 		(net 1)
 	)
-	(via micro
+	(via
 		(at 94.775 39.5)
 		(size 0.6)
@@
 		(net 1)
 	)
-	(via micro
+	(via
 		(at 94.775 40.5)
 		(size 0.6)
@@
 		(net 17)
 	)
-	(via micro
+	(via
 		(at 72.25 79)
 		(size 0.6)
@@
 	)
 	(segment
-		(start 110.279856 77.970144)
-		(end 109.75 77.970144)
+		(start 110.625 77.625)
+		(end 110.279856 77.970144)
 		(width 0.2)
 		(layer "F.Cu")
@@
 	)
 	(segment
-		(start 116.75 77.970144)
-		(end 117.279856 77.970144)
+		(start 110.279856 77.970144)
+		(end 109.75 77.970144)
 		(width 0.2)
 		(layer "F.Cu")
@@
 	(segment
 		(start 117.279856 77.970144)
-		(end 118.25 77)
+		(end 116.75 77.970144)
 		(width 0.2)
 		(layer "F.Cu")
@@
 	)
 	(segment
-		(start 111.25 77)
-		(end 110.279856 77.970144)
+		(start 117.625 77.625)
+		(end 117.279856 77.970144)
 		(width 0.2)
 		(layer "F.Cu")
@@
 	)
 	(via micro
-		(at 111.25 77)
+		(at 110.625 77.625)
 		(size 0.6)
 		(drill 0.3)
-		(layers "F.Cu" "In1.Cu")
+		(layers "F.Cu" "B.Cu")
 		(net 18)
 	)
 	(via micro
-		(at 118.25 77)
+		(at 117.625 77.625)
 		(size 0.6)
 		(drill 0.3)
-		(layers "F.Cu" "In1.Cu")
+		(layers "F.Cu" "B.Cu")
 		(net 18)
 	)
@@
 	)
 	(segment
-		(start 104 75.5)
-		(end 104 58.914215)
+		(start 110 77)
+		(end 105.5 77)
 		(width 0.2)
 		(layer "In1.Cu")
@@
 	)
 	(segment
-		(start 111.25 77)
-		(end 118.25 77)
+		(start 105.4 57.514215)
+		(end 105.4 49.9)
 		(width 0.2)
 		(layer "In1.Cu")
@@
 	)
 	(segment
-		(start 104 58.914215)
-		(end 105.4 57.514215)
+		(start 117.625 77.625)
+		(end 117.25 78)
 		(width 0.2)
 		(layer "In1.Cu")
@@
 	)
 	(segment
-		(start 111.25 77)
-		(end 105.5 77)
+		(start 117.25 78)
+		(end 111 78)
 		(width 0.2)
 		(layer "In1.Cu")
@@
 	)
 	(segment
-		(start 105.4 57.514215)
-		(end 105.4 49.9)
+		(start 104 58.914215)
+		(end 105.4 57.514215)
 		(width 0.2)
 		(layer "In1.Cu")
@@
 	)
 	(segment
+		(start 104 75.5)
+		(end 104 58.914215)
+		(width 0.2)
+		(layer "In1.Cu")
+		(net 18)
+	)
+	(segment
+		(start 110.625 77.625)
+		(end 110 77)
+		(width 0.2)
+		(layer "In1.Cu")
+		(net 18)
+	)
+	(segment
 		(start 105.4 49.9)
 		(end 98.625 43.125)
@@
 	)
 	(segment
+		(start 111 78)
+		(end 110.625 77.625)
+		(width 0.2)
+		(layer "In1.Cu")
+		(net 18)
+	)
+	(segment
 		(start 98.44 76)
 		(end 98.25 76)
@@
 		(polygon
 			(pts
-				(xy 104.75 77) (xy 117.75 77) (xy 117.75 82.5) (xy 117.75 85.5) (xy 144.25 85.5) (xy 144.25 74.5)
-				(xy 144.25 60.5) (xy 104.75 60.5)
+				(xy 104.75 77) (xy 117.75 77) (xy 117.75 82.5) (xy 117.75 85.5) (xy 145 85.5) (xy 145 75) (xy 145 60.5)
+				(xy 104.75 60.5)
 			)
 		)
@@
 		(polygon
 			(pts
-				(xy 98.25 59) (xy 99.25 59) (xy 99.25 55.5) (xy 98.25 54) (xy 98.25 52) (xy 96.75 52) (xy 96.75 55)
+				(xy 98.25 59) (xy 99.25 59) (xy 99.25 55.5) (xy 98.25 54) (xy 98.25 51.5) (xy 96.75 51.5) (xy 96.75 55)
 				(xy 98.25 56)
 			)
